File: schematic/PICerino_TMS9928.sch (KiCad schematic (older format))
At the start: 73 parts, among them CON1 PICERINO-EDGE, IC1 ADG453/413, IC2 AD813ANZ, J1 Conn_01x03, J10 Conn_01x03, J2 Conn_01x03, J3 Conn_01x02, J4 Conn_01x03, J5 Conn_01x03_Yb, J6 Conn_01x03_Y, J7 Conn_01x03_Yr, J8 Conn_01x08, J9 Conn_01x08, U1 LM1881, Y1 Crystal

Commit message: updated board to new zener diode bias design. After testing this provided the best adjustment range. Could use some more work to simply it and check failure conditions.
Parts:
- added R17: 10R, Resistor_THT:R_Axial_DIN0207_L6.3mm_D2.5mm_P7.62mm_Horizontal, symbol Device:R
- added R18: 2R2, Resistor_THT:R_Axial_DIN0207_L6.3mm_D2.5mm_P7.62mm_Horizontal, symbol Device:R
- R16: value 1M -> 47K
- R2: value 470R -> 120R
- RV1: value R_POT -> 100R
Connections:
- net VSS: now also C29.1; no longer C29.2
- net at C14.1, IC1.10 (D3), IC1.15 (D2)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: now also RV1.2; no longer C29.1, R2.1, RV1.1
- new net: R17.1, R18.2, RV1.3
- new net: C29.2, R17.2, R2.1, RV1.1
- new net: D1.1 (K), R18.1
Other:
- moved on the sheet: C29, D1, TP2
Changed lines of the file:
@@
 L Device:D_Zener D1
 U 1 1 62ECC992
-P 4300 9375
-F 0 "D1" V 4254 9455 50  0000 L CNN
-F 1 "D_Zener_2-7" V 4345 9455 50  0000 L CNN
-F 2 "Diode_THT:D_DO-34_SOD68_P7.62mm_Horizontal" H 4300 9375 50  0001 C CNN
-F 3 "~" H 4300 9375 50  0001 C CNN
-	1    4300 9375
-	0    1    1    0
+P 4150 9625
+F 0 "D1" V 4104 9705 50  0000 L CNN
+F 1 "D_Zener_2-7" H 4100 9475 50  0000 L CNN
+F 2 "Diode_THT:D_DO-34_SOD68_P7.62mm_Horizontal" H 4150 9625 50  0001 C CNN
+F 3 "~" H 4150 9625 50  0001 C CNN
+	1    4150 9625
+	-1   0    0    1
 $EndComp
 $Comp
@@
 P 4300 9025
 F 0 "RV1" H 4231 9071 50  0000 R CNN
-F 1 "R_POT" H 4231 8980 50  0000 R CNN
+F 1 "100R" H 4231 8980 50  0000 R CNN
 F 2 "Potentiometer_THT:Potentiometer_Piher_PT-6-V_Vertical" H 4300 9025 50  0001 C CNN
 F 3 "~" H 4300 9025 50  0001 C CNN
@@
 	1    0    0    -1
 $EndComp
-Wire Wire Line
-	4300 9225 4300 9200
-Wire Wire Line
-	4450 9025 4450 9200
-Wire Wire Line
-	4450 9200 4300 9200
-Connection ~ 4300 9200
-Wire Wire Line
-	4300 9200 4300 9175
 $Comp
 L Device:R R2
@@
 P 4125 8700
 F 0 "R2" V 4225 8530 50  0000 L CNN
-F 1 "470R" V 4225 8650 50  0000 L CNN
+F 1 "120R" V 4225 8650 50  0000 L CNN
 F 2 "Resistor_THT:R_Axial_DIN0207_L6.3mm_D2.5mm_P7.62mm_Horizontal" V 4055 8700 50  0001 C CNN
 F 3 "~" H 4125 8700 50  0001 C CNN
@@
 $EndComp
 Wire Wire Line
-	4300 8875 4300 8700
+	4300 8875 4300 8850
 Wire Wire Line
 	4300 8700 4275 8700
@@
 L power:VSS #PWR07
 U 1 1 62F6BAC1
-P 4300 9525
-F 0 "#PWR07" H 4300 9375 50  0001 C CNN
-F 1 "VSS" V 4200 9625 50  0000 C CNN
-F 2 "" H 4300 9525 50  0001 C CNN
-F 3 "" H 4300 9525 50  0001 C CNN
-	1    4300 9525
-	-1   0    0    1
+P 4000 9625
+F 0 "#PWR07" H 4000 9475 50  0001 C CNN
+F 1 "VSS" V 3900 9725 50  0000 C CNN
+F 2 "" H 4000 9625 50  0001 C CNN
+F 3 "" H 4000 9625 50  0001 C CNN
+	1    4000 9625
+	0    -1   -1   0
 $EndComp
 Wire Wire Line
@@
 Wire Wire Line
 	6450 7900 6200 7900
-Wire Wire Line
-	4300 8700 4675 8700
 Connection ~ 4300 8700
 Wire Wire Line
@@
 L Connector:TestPoint TP2
 U 1 1 638CA91D
-P 4675 8700
-F 0 "TP2" H 4617 8726 50  0000 R CNN
-F 1 "TestPoint" H 4617 8817 50  0000 R CNN
-F 2 "Connector_PinHeader_2.54mm:PinHeader_1x01_P2.54mm_Vertical" H 4875 8700 50  0001 C CNN
-F 3 "~" H 4875 8700 50  0001 C CNN
-	1    4675 8700
+P 5625 8800
+F 0 "TP2" H 5567 8826 50  0000 R CNN
+F 1 "TestPoint" H 5567 8917 50  0000 R CNN
+F 2 "Connector_PinHeader_2.54mm:PinHeader_1x01_P2.54mm_Vertical" H 5825 8800 50  0001 C CNN
+F 3 "~" H 5825 8800 50  0001 C CNN
+	1    5625 8800
 	-1   0    0    1
 $EndComp
-Connection ~ 4675 8700
-Wire Wire Line
-	4675 8700 5300 8700
 $Comp
 L Connector:TestPoint TP1
@@
 U 1 1 638F62AC
 P 5300 9125
-F 0 "C14" V 5050 9125 50  0000 C CNN
-F 1 "10uF" V 5166 9125 50  0000 C CNN
+F 0 "C14" H 5450 9175 50  0000 C CNN
+F 1 "10uF" H 5475 9100 50  0000 C CNN
 F 2 "Capacitor_THT:CP_Radial_D5.0mm_P2.50mm" H 5300 9125 50  0001 C CNN
 F 3 "~" H 5300 9125 50  0001 C CNN
@@
 $EndComp
 Wire Wire Line
-	5300 9025 5300 8700
-Connection ~ 5300 8700
-Wire Wire Line
 	5300 8700 5625 8700
 $Comp
@@
 P 5300 9225
 F 0 "#PWR015" H 5300 9075 50  0001 C CNN
-F 1 "VSS" V 5200 9325 50  0000 C CNN
+F 1 "VSS" H 5300 9375 50  0000 C CNN
 F 2 "" H 5300 9225 50  0001 C CNN
 F 3 "" H 5300 9225 50  0001 C CNN
@@
 L Device:C C29
 U 1 1 63BFED24
-P 5625 8850
-F 0 "C29" H 5740 8896 50  0000 L CNN
-F 1 "100nF" H 5740 8805 50  0000 L CNN
-F 2 "Capacitor_THT:C_Disc_D4.7mm_W2.5mm_P5.00mm" H 5663 8700 50  0001 C CNN
-F 3 "~" H 5625 8850 50  0001 C CNN
-	1    5625 8850
-	1    0    0    -1
+P 4825 8700
+F 0 "C29" V 4700 8625 50  0000 L CNN
+F 1 "100nF" V 4975 8625 50  0000 L CNN
+F 2 "Capacitor_THT:C_Disc_D4.7mm_W2.5mm_P5.00mm" H 4863 8550 50  0001 C CNN
+F 3 "~" H 4825 8700 50  0001 C CNN
+	1    4825 8700
+	0    1    1    0
 $EndComp
 Connection ~ 5625 8700
@@
 L power:VSS #PWR0101
 U 1 1 63BFF3BC
-P 5625 9000
-F 0 "#PWR0101" H 5625 8850 50  0001 C CNN
-F 1 "VSS" V 5525 9100 50  0000 C CNN
-F 2 "" H 5625 9000 50  0001 C CNN
-F 3 "" H 5625 9000 50  0001 C CNN
-	1    5625 9000
-	-1   0    0    1
+P 4975 8700
+F 0 "#PWR0101" H 4975 8550 50  0001 C CNN
+F 1 "VSS" V 4875 8800 50  0000 C CNN
+F 2 "" H 4975 8700 50  0001 C CNN
+F 3 "" H 4975 8700 50  0001 C CNN
+	1    4975 8700
+	0    1    1    0
 $EndComp
 Wire Wire Line
@@
 U 1 1 62AB4DAE
 P 6200 8850
-F 0 "R16" V 6300 8775 50  0000 L CNN
-F 1 "1M" V 6100 8800 50  0000 L CNN
+F 0 "R16" H 6000 8775 50  0000 L CNN
+F 1 "47K" H 6000 8875 50  0000 L CNN
 F 2 "Resistor_THT:R_Axial_DIN0207_L6.3mm_D2.5mm_P7.62mm_Horizontal" V 6130 8850 50  0001 C CNN
 F 3 "~" H 6200 8850 50  0001 C CNN
@@
 P 6200 9000
 F 0 "#PWR0102" H 6200 8850 50  0001 C CNN
-F 1 "VSS" V 6275 9100 50  0000 C CNN
+F 1 "VSS" H 6200 9175 50  0000 C CNN
 F 2 "" H 6200 9000 50  0001 C CNN
 F 3 "" H 6200 9000 50  0001 C CNN
@@
 Wire Wire Line
 	7550 7150 11375 7150
+Wire Wire Line
+	4300 9175 4300 9225
+Wire Wire Line
+	4300 8850 3850 8850
+Wire Wire Line
+	3850 8850 3850 8900
+Connection ~ 4300 8850
+Wire Wire Line
+	4300 8850 4300 8700
+Wire Wire Line
+	3850 9200 3850 9225
+Wire Wire Line
+	3850 9225 4300 9225
+$Comp
+L Device:R R18
+U 1 1 62C0EF92
+P 4300 9375
+F 0 "R18" H 4150 9350 50  0000 L CNN
+F 1 "2R2" H 4100 9425 50  0000 L CNN
+F 2 "Resistor_THT:R_Axial_DIN0207_L6.3mm_D2.5mm_P7.62mm_Horizontal" V 4230 9375 50  0001 C CNN
+F 3 "~" H 4300 9375 50  0001 C CNN
+	1    4300 9375
+	-1   0    0    1
+$EndComp
+Connection ~ 4300 9225
+Wire Wire Line
+	4300 9625 4300 9525
+$Comp
+L Device:R R17
+U 1 1 62B66C19
+P 3850 9050
+F 0 "R17" H 3975 9025 50  0000 L CNN
+F 1 "10R" H 3925 9125 50  0000 L CNN
+F 2 "Resistor_THT:R_Axial_DIN0207_L6.3mm_D2.5mm_P7.62mm_Horizontal" V 3780 9050 50  0001 C CNN
+F 3 "~" H 3850 9050 50  0001 C CNN
+	1    3850 9050
+	-1   0    0    1
+$EndComp
+Wire Wire Line
+	5300 8700 5300 9025
+Connection ~ 5300 9025
+Wire Wire Line
+	5625 8800 5625 8700
 Wire Bus Line
 	13700 2350 13700 3900
@@
 Wire Bus Line
 	3500 3550 3500 4250
+Wire Wire Line
+	4300 8700 4675 8700
+Wire Wire Line
+	4450 9025 5300 9025
 $EndSCHEMATC

Commit message: updated variable capacitor pads to be a bit larger
Other:
- note added: "RAM DEBUG PORTS"
Changed lines of the file:
@@
 Wire Wire Line
 	5625 8800 5625 8700
+Wire Wire Line
+	4300 8700 4675 8700
+Wire Wire Line
+	4450 9025 5300 9025
 Wire Bus Line
 	13700 2350 13700 3900
@@
 Wire Bus Line
 	3500 3550 3500 4250
-Wire Wire Line
-	4300 8700 4675 8700
-Wire Wire Line
-	4450 9025 5300 9025
+Text Notes 15400 1575 0    50   ~ 0
+RAM DEBUG PORTS
 $EndSCHEMATC
