File: schematic/PICerino_TMS9928.kicad_sch (KiCad schematic)
At the start: 76 parts, among them CON1 PICERINO-EDGE, IC1 ADG453/413, IC2 AD813ANZ, J1 Conn_01x03, J10 Conn_01x03, J2 Conn_01x03, J3 Conn_01x02, J4 Conn_01x03, J5 Conn_01x03_Yb, J6 Conn_01x03_Y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

Commit message: added mit license to hardware
Other:
- company: (none) -> sparkletron
- title: (none) -> TMS99XX
Changed lines of the file:
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@@
 (kicad_sch (version 20211123) (generator eeschema)
   (paper "B")
+  (title_block
+    (title "TMS99XX")
+    (company "sparkletron")
+    (comment 1 "Jay Converitno")
+    (comment 2 "MIT License")
+  )
   (junction (at 294.64 99.06) (diameter 0) (color 0 0 0 0)
   )
